File: RotaryEncoder.kicad_pcb (KiCad board)
At the start: 2 copper layers, 20 x 28 mm, 9 parts, among them J1 Conn_01x04, J2 Conn_01x02

Commit message: Add manufacturing data
Parts:
- added G***: OSHW_LOGO_5MM, dresco:OSHW_LOGO_5MM, F.Cu at (134.0, 114.5)
- turned C1 to 90 degrees
- turned C2 to 90 degrees
- turned R1 to 90 degrees
- turned R2 to 90 degrees
- turned R3 to 90 degrees
- turned R4 to 90 degrees
Routing:
- net GND: track 0.00 -> 36.5 mm, vias 0 -> 2
- net VCC: track 0.00 -> 16.3 mm
- net B: track 0.00 -> 13.5 mm
- net A: track 0.00 -> 10.5 mm
- net B1: track 0.00 -> 7.80 mm
- net A1: track 0.00 -> 7.78 mm
- net SW2: track 0.00 -> 4.92 mm
- net SW1: track 0.00 -> 4.92 mm
- added copper zone on B.Cu, net GND
Other:
- outline, holes or cut-outs redrawn
- board text added: "-GND -VCC -B -A"
- board text added: "CC-BY-SA"
- board text added: "PEC11R breakout v1.00 github.com/dresco"
- board text added: "SW1- SW2-"
- board text removed: "-GND- -VCC- -B- -A-"
